Commit message: sort of works with cylinder. debugging contact

File: drake/examples/kuka_iiwa_arm/models/objects/simple_cuboid.urdf (robot description, URDF)
Before this commit: robot simple_cuboid, 1 links, 0 joints
Links:
- link base_link: mass 0.5 -> 0.1; geometry collision box size=0.06 0.06 0.2; visual box size=0.06 0.06 0.2
