Commit message: moving to two arm

File: drake/manipulation/models/iiwa_description/urdf/iiwa14_polytope_collision_ball_flange_collision.urdf (robot description, URDF)
Before this commit: robot iiwa14, 11 links, 10 joints
Links:
- link iiwa_link_7: geometry visual mesh filename=../meshes/visual/link_7.obj
- link iiwa_link_ee: geometry collision sphere radius=0.0; collision sphere radius=0.0
