Commit message: updated configurations

File: drake/manipulation/models/iiwa_description/urdf/sfeng_dual_iiwa14_polytope_collision.urdf (robot description, URDF)
Before this commit: robot dual_iiwa14, 21 links, 19 joints
Joints:
- joint left_iiwa_base_joint: origin xyz=1.86 0 0 rpy=0 0 3.1415926 -> xyz=1.28 0 0 rpy=0 0 3.1415926
