Commit message: Mesh updates for fetch + floating-base (#1)
* Replace dae extensions with obj in fetch.urdf

* Add blank material files for links converted from STL

* Use floating base in passive demo

* Make l_gripper_finger_link.obj.mtl blank

File: drake/examples/Fetch/fetch_description/robots/fetch.urdf (robot description, URDF)
Before this commit: robot fetch, 26 links, 25 joints
Links:
- link base_link: geometry collision mesh filename=../meshes/base_link_collision.obj; visual mesh filename=../meshes/base_link.obj
- link elbow_flex_link: geometry collision mesh filename=../meshes/elbow_flex_link_collision.obj; visual mesh filename=../meshes/elbow_flex_link.obj
- link forearm_roll_link: geometry collision mesh filename=../meshes/forearm_roll_link_collision.obj; visual mesh filename=../meshes/forearm_roll_link.obj
- link gripper_link: geometry collision mesh filename=../meshes/gripper_link.obj; visual mesh filename=../meshes/gripper_link.obj
- link head_pan_link: geometry collision mesh filename=../meshes/head_pan_link_collision.obj; visual mesh filename=../meshes/head_pan_link.obj
- link head_tilt_link: geometry collision mesh filename=../meshes/head_tilt_link_collision.obj; visual mesh filename=../meshes/head_tilt_link.obj
- link shoulder_lift_link: geometry collision mesh filename=../meshes/shoulder_lift_link_collision.obj; visual mesh filename=../meshes/shoulder_lift_link.obj
- link shoulder_pan_link: geometry collision mesh filename=../meshes/shoulder_pan_link_collision.obj; visual mesh filename=../meshes/shoulder_pan_link.obj
- link torso_fixed_link: geometry collision mesh filename=../meshes/torso_fixed_link.obj; visual mesh filename=../meshes/torso_fixed_link.obj
- link torso_lift_link: geometry collision mesh filename=../meshes/torso_lift_link_collision.obj; visual mesh filename=../meshes/torso_lift_link.obj
- link upperarm_roll_link: geometry collision mesh filename=../meshes/upperarm_roll_link_collision.obj; visual mesh filename=../meshes/upperarm_roll_link.obj
- link wrist_flex_link: geometry collision mesh filename=../meshes/wrist_flex_link_collision.obj; visual mesh filename=../meshes/wrist_flex_link.obj
- link wrist_roll_link: geometry collision mesh filename=../meshes/wrist_roll_link_collision.obj; visual mesh filename=../meshes/wrist_roll_link.obj

Commit message: Tuned contact stiffness, removed belows links, cleaned up file names, and added urdf license text file.

File: drake/examples/Fetch/fetch_description/robots/fetch.urdf (robot description, URDF)
Before this commit: robot fetch, 26 links, 25 joints
Links:
- removed link bellows_link
- removed link bellows_link2
Joints:
- removed joint bellows_joint
- removed joint bellows_joint2

Commit message: init add

File: drake/examples/Fetch/fetch_description/robots/fetch.urdf (robot description, URDF)
Before this commit: robot fetch, 24 links, 23 joints
Links:
- link torso_lift_link: geometry visual mesh filename=../meshes/torso_lift_link.obj

Commit message: added ball joints

File: drake/examples/Fetch/fetch_description/robots/fetch.urdf (robot description, URDF)
Before this commit: robot fetch, 24 links, 23 joints
Links:
- added link back_left_caster, mass 0.1; collision sphere radius=0.02; visual sphere radius=0.02
- added link back_right_caster, mass 0.1; collision sphere radius=0.02; visual sphere radius=0.02
- added link front_left_caster, mass 0.1; collision sphere radius=0.02; visual sphere radius=0.02
- added link front_right_caster, mass 0.1; collision sphere radius=0.02; visual sphere radius=0.02
- link base_link: geometry visual mesh filename=../meshes/base_link.obj
Joints:
- added joint back_left_caster_ball_joint: type ball, parent base_link, child back_left_caster, origin xyz=-0.21 0.12 0.01 rpy=0 0 0
- added joint back_right_caster_ball_joint: type ball, parent base_link, child back_right_caster, origin xyz=-0.21 -0.12 0.01 rpy=0 0 0
- added joint front_left_caster_ball_joint: type ball, parent base_link, child front_left_caster, origin xyz=0.17 0.12 0.01 rpy=0 0 0
- added joint front_right_caster_ball_joint: type ball, parent base_link, child front_right_caster, origin xyz=0.17 -0.12 0.01 rpy=0 0 0
